File: hardware/chademo-charge-controller/chademo-charge-controller.kicad_sch (KiCad schematic)
At the start: 26 parts, among them IC1 TPS62160DGKR, IC2 MCP2515-I_ST, IC3 SN65HVD230, IC4 MCP2515-I_ST, IC5 SN65HVD230, IC6 NCV8402ASTT1G, J1 M22-2510346, U1 Pico, U2 PC817, U3 PC817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

Commit message: pcb layout, 56pin socket
Parts:
- added J2: Conn_2Rows-57Pins, Connector:delphi56, symbol Connector_Generic:Conn_2Rows-57Pins
- J1: footprint Connector_PinHeader_2.54mm:PinHeader_1x03_P2.54mm_Vertical -> Connector_PinHeader_2.54mm:PinHeader_1x03_P2.54mm_Horizontal
Connections:
- net 12V: now also J2.15 (Pin_15)
- net CP: now also J2.4 (Pin_4)
- net CP2: now also J2.5 (Pin_5)
- net CP3: now also J2.2 (Pin_2)
- net GND: now also J2.1 (Pin_1)
- net OUT2: now also J2.3 (Pin_3)
- net CHARGE_ENABLE renamed OUT_1_CHARGE_ENABLE
- net OUT_1_CHARGE_ENABLE: now also U1.16 (GPIO12); no longer U1.17 (GPIO13)
- net CONTACTOR_ENABLE renamed OUT_2_CONTACTOR_ENABLE
- net OUT_2_CONTACTOR_ENABLE: now also U1.17 (GPIO13); no longer U1.16 (GPIO12)

Commit message: tweaking hw
Parts:
- added D2, D3, D4, D5: LED, LED_SMD:LED_0805_2012Metric, symbol Device:LED
- added R10: 1k, Resistor_SMD:R_0805_2012Metric, symbol Device:R
- added R11, R8, R9: 50, Resistor_SMD:R_0805_2012Metric, symbol Device:R
- R5: value 1k -> 50
Connections:
- net 12V: now also D1.2; no longer C1.1, IC1.2 (VIN), IC1.3 (EN)
- net 3V: now also R10.1, R11.1, R8.1, R9.1
- net 5V: now also U1.39 (VSYS); no longer D1.2
- net CHADEMO_CAN_H: now also J2.23 (Pin_23)
- net CHADEMO_CAN_L: now also J2.51 (Pin_51)
- net GND: now also J2.28 (Pin_28), J2.43 (Pin_43), J2.57 (Pin_57)
- net IN1: now also D2.1 (K)
- net IN2: now also D3.1 (K), R10.2; no longer R5.2
- net MAIN_CAN_H: now also J2.21 (Pin_21)
- net MAIN_CAN_L: now also J2.49 (Pin_49)
- net OUT2: now also D5.1 (K)
- net at D1.1: now also C1.1, IC1.2 (VIN), IC1.3 (EN); no longer U1.39 (VSYS)
- net at R6.2, U4.4: now also D4.1 (K)
- new net: D5.2 (A), R11.2
- new net: D2.2 (A), R5.2
- new net: D4.2 (A), R9.2
- new net: D3.2 (A), R8.2
Other:
- moved on the sheet: IC6, R4, R6

Commit message: lots of work on hardware
Parts:
- added C7: 10uF, Capacitor_SMD:C_0603_1608Metric, symbol Device:C_Small
- added D6, D7, D8: LED, LED_SMD:LED_0805_2012Metric, symbol Device:LED
- added H1, H2: MountingHole_Pad, MountingHole:MountingHole_3.2mm_M3_DIN965_Pad, symbol Mechanical:MountingHole_Pad
- added J3, J7, J8: Conn_01x02_Pin, Connector_PinHeader_2.54mm:PinHeader_1x02_P2.54mm_Vertical, symbol Connector:Conn_01x02_Pin
- added JP1, JP2: SolderJumper_2_Open, Jumper:SolderJumper-2_P1.3mm_Open_Pad1.0x1.5mm, symbol Jumper:SolderJumper_2_Open
- added R12, R13: 120, Resistor_SMD:R_0805_2012Metric, symbol Device:R_US
- added R14, R16, R21: 1k, Resistor_SMD:R_0805_2012Metric, symbol Device:R
- added R15, R20, R23: 50, Resistor_SMD:R_0805_2012Metric, symbol Device:R
- added R17, R18, R19: 560, Resistor_SMD:R_0805_2012Metric, symbol Device:R
- added R22: 100, Resistor_SMD:R_0805_2012Metric, symbol Device:R
- added U5, U6, U7: PC817, Package_DIP:DIP-4_W7.62mm, symbol Isolator:PC817
Connections:
- net 12V: now also C1.1, D1.1, IC1.2 (VIN), IC1.3 (EN), J2.33 (Pin_33), J2.9 (Pin_9), D8.1 (K), R17.1, U5.1, U7.4; no longer D1.2, J2.15 (Pin_15)
- net 3V: now also R15.1, R16.1, R20.1, R21.1, R23.1
- net 5V: now also J7.2 (Pin_2)
- net CHADEMO_CAN_H: now also J8.2 (Pin_2), R13.1
- net CHADEMO_CAN_L: now also J2.22 (Pin_22), J8.1 (Pin_1), JP2.2 (B); no longer J2.51 (Pin_51)
- net CP2: now also C6.2, IC6.3 (S), U3.2; no longer C6.1, U3.1
- net GND: now also J2.42 (Pin_42), J2.56 (Pin_56), C7.2, H1.1, H2.1, J7.1 (Pin_1), U5.3, U6.2, U6.3, U7.2; no longer C6.2, IC6.3 (S), J2.28 (Pin_28), U3.2
- net MAIN_CAN_H: now also J3.2 (Pin_2), R12.1
- net MAIN_CAN_L: now also J2.20 (Pin_20), J3.1 (Pin_1), JP1.2 (B); no longer J2.49 (Pin_49)
- net OUT2: no longer D5.1 (K), IC6.2 (D_1)
- net CHARGE_ENABLE: now reaches J2.12 (Pin_12)
- net CHARGE_ENABLE: now also U7.3
- net CONCTACTOR_POS: now reaches J2.32 (Pin_32)
- net CONCTACTOR_POS: now also J2.4 (Pin_4), R18.1
- net PROX: now reaches J2.36 (Pin_36)
- net PROX: now also R14.2
- net CHARGE_INHIBIT: now reaches J2.7 (Pin_7)
- net CHARGE_INHIBIT: now also R19.1
- net MANUAL_WAKE_SWITCH_A: now reaches J2.8 (Pin_8)
- net MANUAL_WAKE_SWITCH_A: now also U1.15 (GPIO11), D6.1 (K), R16.2, U5.4
- net CHARGE_ENABLE_MCU: now reaches U1.12 (GPIO9)
- net CHARGE_ENABLE_MCU: now also R22.1
- net CHARGE_INHIBIT_MCU: now reaches U1.14 (GPIO10)
- net CHARGE_INHIBIT_MCU: now also D7.1 (K), R21.2, U6.4
- net CP: no longer names the net of C5.1, U2.1
- net CP: now also R18.2; no longer J2.4 (Pin_4)
- net WAKE: no longer names the net of U1.29 (GPIO22)
- new net: C6.1, R17.2, U3.1
- new net: JP1.1 (A), R12.2
- new net: D7.2 (A), R20.2
- new net: C7.1, R19.2, U6.1
- new net: R14.1, U5.2
- new net: D6.2 (A), R15.2
- new net: R22.2, U7.1
- new net: JP2.1 (A), R13.2
- new net: D8.2 (A), R23.2
- new net 12V_IN: D1.2, J2.15 (Pin_15)
- new net CONTACTOR_NEG: D5.1 (K), IC6.2 (D_1)
Other:
- note added: "Charge enable output signal"
- note added: "Charge inhibit input"
- note added: "Proximity"
- moved on the sheet: C1, C2, C3, C4, C5, C6, D1, D2, D3, D4, D5, IC1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

Commit message: I dunno ... lots
Parts:
- R10, R16, R21, R4: value 1k -> 1k6
- R11, R15, R20, R23, R5, R8, R9: value 50 -> 10
Connections:
- net OUT2 is gone; now on net CONTACTOR_NEG: J2.3 (Pin_3)
- net 12V: no longer D8.1 (K)
- net 3V: no longer R23.1
- net CHARGE_ENABLE_MCU: now also R23.1
- net GND: now also D8.1 (K)
Other:
- moved on the sheet: D8, R23
Changed lines of the file:
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@@
   (junction (at 220.98 264.16) (diameter 0) (color 0 0 0 0)
   )
+  (junction (at 179.07 372.11) (diameter 0) (color 0 0 0 0)
+  )
   (junction (at 144.78 55.88) (diameter 0) (color 0 0 0 0)
   )
+  (junction (at 179.07 389.89) (diameter 0) (color 0 0 0 0)
+  )
   (junction (at 401.32 88.9) (diameter 0) (color 0 0 0 0)
   )
@@
   (junction (at 392.43 175.26) (diameter 0) (color 0 0 0 0)
   )
-  (junction (at 219.71 384.81) (diameter 0) (color 0 0 0 0)
-  )
   (junction (at 172.72 204.47) (diameter 0) (color 0 0 0 0)
   )
@@
     (stroke (width 0) (type default))
   )
-  (wire (pts (xy 189.23 372.11) (xy 193.04 372.11))
+  (wire (pts (xy 173.99 372.11) (xy 179.07 372.11))
     (stroke (width 0) (type default))
   )
@@
     (stroke (width 0) (type default))
   )
+  (wire (pts (xy 179.07 389.89) (xy 201.93 389.89))
+    (stroke (width 0) (type default))
+  )
   (wire (pts (xy 220.98 334.01) (xy 212.09 334.01))
     (stroke (width 0) (type default))
@@
     (stroke (width 0) (type default))
   )
-  (wire (pts (xy 219.71 382.27) (xy 219.71 384.81))
-    (stroke (width 0) (type default))
-  )
   (wire (pts (xy 55.88 55.88) (xy 55.88 48.26))
     (stroke (width 0) (type default))
@@
     (stroke (width 0) (type default))
   )
+  (wire (pts (xy 179.07 388.62) (xy 179.07 389.89))
+    (stroke (width 0) (type default))
+  )
   (wire (pts (xy 123.19 170.18) (xy 116.84 170.18))
     (stroke (width 0) (type default))
@@
     (stroke (width 0) (type default))
   )
-  (wire (pts (xy 219.71 384.81) (xy 217.17 384.81))
-    (stroke (width 0) (type default))
-  )
   (wire (pts (xy 392.43 175.26) (xy 379.73 175.26))
     (stroke (width 0) (type default))
@@
     (stroke (width 0) (type default))
   )
+  (wire (pts (xy 179.07 373.38) (xy 179.07 372.11))
+    (stroke (width 0) (type default))
+  )
   (wire (pts (xy 209.55 259.08) (xy 220.98 259.08))
     (stroke (width 0) (type default))
@@
     (stroke (width 0) (type default))
   )
-  (wire (pts (xy 219.71 365.76) (xy 237.49 365.76))
-    (stroke (width 0) (type default))
-  )
   (wire (pts (xy 405.13 134.62) (xy 403.86 134.62))
     (stroke (width 0) (type default))
@@
     (stroke (width 0) (type default))
   )
+  (wire (pts (xy 179.07 372.11) (xy 193.04 372.11))
+    (stroke (width 0) (type default))
+  )
   (wire (pts (xy 228.6 87.63) (xy 233.68 87.63))
     (stroke (width 0) (type default))
@@
     (stroke (width 0) (type default))
   )
-  (wire (pts (xy 189.23 389.89) (xy 201.93 389.89))
+  (wire (pts (xy 168.91 389.89) (xy 179.07 389.89))
     (stroke (width 0) (type default))
   )
@@
     (stroke (width 0) (type default))
   )
-  (wire (pts (xy 232.41 384.81) (xy 219.71 384.81))
-    (stroke (width 0) (type default))
-  )
-  (wire (pts (xy 219.71 365.76) (xy 219.71 367.03))
+  (wire (pts (xy 217.17 384.81) (xy 232.41 384.81))
     (stroke (width 0) (type default))
   )
@@
     )
   )
-  (global_label "CHARGE_ENABLE_MCU" (shape input) (at 189.23 372.11 180) (fields_autoplaced)
+  (global_label "CHARGE_ENABLE_MCU" (shape input) (at 173.99 372.11 180) (fields_autoplaced)
     (effects (font (size 1.27 1.27)) (justify right))
-    (property "Intersheetrefs" "${INTERSHEET_REFS}" (at 165.9438 372.11 0)
+    (property "Intersheetrefs" "${INTERSHEET_REFS}" (at 150.7038 372.11 0)
       (effects (font (size 1.27 1.27)) (justify right) hide)
     )
@@
     )
   )
-  (global_label "GND" (shape output) (at 189.23 389.89 180) (fields_autoplaced)
+  (global_label "GND" (shape output) (at 168.91 389.89 180) (fields_autoplaced)
     (effects (font (size 1.27 1.27)) (justify right))
-    (property "Intersheetrefs" "${INTERSHEET_REFS}" (at 182.4537 389.89 0)
+    (property "Intersheetrefs" "${INTERSHEET_REFS}" (at 162.1337 389.89 0)
       (effects (font (size 1.27 1.27)) (justify right) hide)
     )
@@
     )
   )
-  (global_label "3V" (shape input) (at 237.49 365.76 0) (fields_autoplaced)
-    (effects (font (size 1.27 1.27)) (justify left))
-    (property "Intersheetrefs" "${INTERSHEET_REFS}" (at 242.6939 365.76 0)
-      (effects (font (size 1.27 1.27)) (justify left) hide)
-    )
-  )
   (global_label "CHARGE_ENABLE_MCU" (shape output) (at 74.93 160.02 180) (fields_autoplaced)
     (effects (font (size 1.27 1.27)) (justify right))
@@
     )
   )
-  (global_label "OUT2" (shape input) (at 279.4 50.8 180) (fields_autoplaced)
+  (global_label "CONTACTOR_NEG" (shape input) (at 279.4 50.8 180) (fields_autoplaced)
     (effects (font (size 1.27 1.27)) (justify right))
-    (property "Intersheetrefs" "${INTERSHEET_REFS}" (at 271.6561 50.8 0)
+    (property "Intersheetrefs" "${INTERSHEET_REFS}" (at 260.9518 50.8 0)
       (effects (font (size 1.27 1.27)) (justify right) hide)
     )
@@
       (effects (font (size 1.27 1.27)) (justify left))
     )
-    (property "Value" "1k" (at 230.378 53.213 0)
+    (property "Value" "1k6" (at 230.378 53.213 0)
       (effects (font (size 1.27 1.27)) (justify left))
     )
@@
       (effects (font (size 1.27 1.27)) (justify left))
     )
-    (property "Value" "1k" (at 230.378 323.723 0)
+    (property "Value" "1k6" (at 230.378 323.723 0)
       (effects (font (size 1.27 1.27)) (justify left))
     )
@@
       (effects (font (size 1.27 1.27)) (justify left))
     )
-    (property "Value" "50" (at 217.678 45.593 0)
+    (property "Value" "10" (at 217.678 45.593 0)
       (effects (font (size 1.27 1.27)) (justify left))
     )
@@
       (effects (font (size 1.27 1.27)) (justify left))
     )
-    (property "Value" "50" (at 216.408 140.843 0)
+    (property "Value" "10" (at 216.408 140.843 0)
       (effects (font (size 1.27 1.27)) (justify left))
     )
@@
       (effects (font (size 1.27 1.27)) (justify left))
     )
-    (property "Value" "50" (at 198.628 246.253 0)
+    (property "Value" "10" (at 198.628 246.253 0)
       (effects (font (size 1.27 1.27)) (justify left))
     )
@@
       (effects (font (size 1.27 1.27)) (justify left))
     )
-    (property "Value" "1k" (at 230.378 101.473 0)
+    (property "Value" "1k6" (at 230.378 101.473 0)
       (effects (font (size 1.27 1.27)) (justify left))
     )
@@
       (effects (font (size 1.27 1.27)) (justify left))
     )
-    (property "Value" "50" (at 217.678 316.103 0)
+    (property "Value" "10" (at 217.678 316.103 0)
       (effects (font (size 1.27 1.27)) (justify left))
     )
@@
       (effects (font (size 1.27 1.27)) (justify left))
     )
-    (property "Value" "50" (at 174.498 187.833 0)
+    (property "Value" "10" (at 174.498 187.833 0)
       (effects (font (size 1.27 1.27)) (justify left))
     )
@@
     )
   )
-  (symbol (lib_id "Device:R") (at 219.71 370.84 0) (unit 1)
+  (symbol (lib_id "Device:R") (at 179.07 377.19 0) (unit 1)
     (in_bom yes) (on_board yes) (dnp no)
-    (property "Reference" "R23" (at 221.488 369.6716 0)
+    (property "Reference" "R23" (at 180.848 376.0216 0)
       (effects (font (size 1.27 1.27)) (justify left))
     )
-    (property "Value" "50" (at 221.488 371.983 0)
+    (property "Value" "10" (at 180.848 378.333 0)
       (effects (font (size 1.27 1.27)) (justify left))
     )
-    (property "Footprint" "Resistor_SMD:R_0805_2012Metric" (at 217.932 370.84 90)
+    (property "Footprint" "Resistor_SMD:R_0805_2012Metric" (at 177.292 377.19 90)
       (effects (font (size 1.27 1.27)) hide)
     )
-    (property "Datasheet" "~" (at 219.71 370.84 0)
+    (property "Datasheet" "~" (at 179.07 377.19 0)
       (effects (font (size 1.27 1.27)) hide)
     )
@@
       (effects (font (size 1.27 1.27)) (justify left))
     )
-    (property "Value" "1k" (at 211.328 253.873 0)
+    (property "Value" "1k6" (at 211.328 253.873 0)
       (effects (font (size 1.27 1.27)) (justify left))
     )
@@
     )
   )
-  (symbol (lib_id "Device:LED") (at 219.71 378.46 90) (unit 1)
+  (symbol (lib_id "Device:LED") (at 179.07 384.81 90) (unit 1)
     (in_bom yes) (on_board yes) (dnp no) (fields_autoplaced)
-    (property "Reference" "D8" (at 223.52 379.4125 90)
+    (property "Reference" "D8" (at 182.88 385.7625 90)
       (effects (font (size 1.27 1.27)) (justify right))
     )
-    (property "Value" "LED" (at 223.52 381.9525 90)
+    (property "Value" "LED" (at 182.88 388.3025 90)
       (effects (font (size 1.27 1.27)) (justify right))
     )
-    (property "Footprint" "LED_SMD:LED_0805_2012Metric" (at 219.71 378.46 0)
+    (property "Footprint" "LED_SMD:LED_0805_2012Metric" (at 179.07 384.81 0)
       (effects (font (size 1.27 1.27)) hide)
     )
-    (property "Datasheet" "~" (at 219.71 378.46 0)
+    (property "Datasheet" "~" (at 179.07 384.81 0)
       (effects (font (size 1.27 1.27)) hide)
     )
@@
       (effects (font (size 1.27 1.27)) (justify left))
     )
-    (property "Value" "50" (at 217.678 93.853 0)
+    (property "Value" "10" (at 217.678 93.853 0)
       (effects (font (size 1.27 1.27)) (justify left))
     )
